Commit message: Fixed material name

File: src/ur5/ur5_description/urdf/ur5_robotiq85_gripper.urdf.xacro (robot description, xacro)
@@ -11,5 +11,4 @@
         <mesh filename="package://robotiq_description/meshes/robotiq_85_coupler.stl" />
       </geometry>
-      <material name="flat_black"/>
     </visual>
     <collision>
